Commit message: feat: integrate moveit configuration for indomitus_arm

File: src/arm_description/urdf/arm_macro.xacro (robot description, xacro)
@@ -31,5 +31,5 @@
       <origin xyz="0 0 0.018" rpy="0 0 0"/>
       <axis xyz="0 0 1"/>
-      <limit lower="${-pi}" upper="${pi}" effort="100" velocity="1"/>
+      <limit lower="${-pi}" upper="${pi}" effort="100.0" velocity="1.0"/>
     </joint>
     <link name="arm_base_link">
@@ -47,5 +47,5 @@
       <origin xyz="0 0.013 0.0945" rpy="0 0 ${-pi/2}"/>
       <axis xyz="1 0 0"/>
-      <limit lower="${-pi/2}" upper="${pi}" effort="100" velocity="1"/>
+      <limit lower="${-pi/2}" upper="${pi}" effort="100.0" velocity="1.0"/>
     </joint>
     <link name="arm_shoulder_link">
@@ -63,5 +63,5 @@
       <origin xyz="-0.057 0 0.5" rpy="0 0 0"/>
       <axis xyz="1 0 0"/>
-      <limit lower="${-pi/2}" upper="${pi/2}" effort="100" velocity="1"/>
+      <limit lower="${-pi/2}" upper="${pi/2}" effort="100.0" velocity="1.0"/>
     </joint>
     <link name="arm_forearm_link">
@@ -79,5 +79,5 @@
       <origin xyz="0.002175 0 0.4" rpy="${pi} ${pi} 0"/>
       <axis xyz="1 0 0"/>
-      <limit lower="${-pi/2}" upper="${pi/2}" effort="100" velocity="1"/>
+      <limit lower="${-pi/2}" upper="${pi/2}" effort="100.0" velocity="1.0"/>
     </joint>
     <link name="arm_wrist_1_link">
@@ -95,5 +95,5 @@
       <origin xyz="-0.067825 0 0.0353" rpy="0 ${pi/2} 0"/>
       <axis xyz="1 0 0"/>
-      <limit lower="${-pi}" upper="${pi}" effort="100" velocity="1"/>
+      <limit lower="${-pi}" upper="${pi}" effort="100.0" velocity="1.0"/>
     </joint>
     <link name="arm_wrist_2_link">
@@ -106,10 +106,20 @@
       <xacro:dummy_inertia mass="0.3"/>
     </link>
+    <joint name="arm_wrist_2_end_effector_joint" type="revolute">
+      <parent link="arm_wrist_2_link"/>
+      <child link="arm_end_effector_link"/>
+      <origin xyz="0 0 0.05" rpy="0 0 0"/>
+      <axis xyz="0 0 1"/>
+      <limit lower="${-pi}" upper="${pi}" effort="100.0" velocity="1.0"/>
+    </joint>
+    <link name="arm_end_effector_link">
+      <xacro:dummy_inertia mass="0.2"/>
+    </link>
     <joint name="arm_tcp_joint" type="fixed">
-      <parent link="arm_wrist_2_link"/>
+      <parent link="arm_end_effector_link"/>
       <child link="arm_tcp_link"/>
-      <origin xyz="0 0 0" rpy="0 0 0"/>
+      <origin xyz="0 0 0.02" rpy="0 0 0"/>
     </joint>
-    <!-- TCP (Tool Center Point) is a virtual point, it has no mass or collisions -->
+    <!-- TCP (Tool Center Point) is a virtual point -->
     <link name="arm_tcp_link"/>
   </xacro:macro>

Commit message: feat: integrate ros2_control and fix controller interfaces

File: src/arm_description/urdf/arm_macro.xacro (robot description, xacro)
@@ -123,4 +123,26 @@
     <!-- TCP (Tool Center Point) is a virtual point -->
     <link name="arm_tcp_link"/>
+    <!-- ROS 2 Control Configuration -->
+    <ros2_control name="ArmSystem" type="system">
+      <hardware>
+        <plugin>mock_components/GenericSystem</plugin>
+      </hardware>
+      <xacro:macro name="arm_joint_control" params="joint_name">
+        <joint name="${joint_name}">
+          <command_interface name="position">
+            <param name="min">${-pi}</param>
+            <param name="max">${pi}</param>
+          </command_interface>
+          <state_interface name="position"/>
+          <state_interface name="velocity"/>
+        </joint>
+      </xacro:macro>
+      <xacro:arm_joint_control joint_name="arm_mount_base_joint"/>
+      <xacro:arm_joint_control joint_name="arm_base_shoulder_joint"/>
+      <xacro:arm_joint_control joint_name="arm_shoulder_forearm_joint"/>
+      <xacro:arm_joint_control joint_name="arm_forearm_wrist_1_joint"/>
+      <xacro:arm_joint_control joint_name="arm_wrist_1_wrist_2_joint"/>
+      <xacro:arm_joint_control joint_name="arm_wrist_2_end_effector_joint"/>
+    </ros2_control>
   </xacro:macro>
 </robot>
